File: videoamp/videoamp.sch (KiCad schematic (older format))
At the start: 20 parts, among them J5V1 Conn_01x01, U1 THS7316, U2 AMS1117-3.3

Commit message: Redesign board to provide luma/chroma/composite signals on A/V out
Parts:
- removed JSELECT1: Conn_01x03, Connector_PinHeader_2.54mm:PinHeader_1x03_P2.54mm_Horizontal, symbol Connector_Generic:Conn_01x03
- added JAV6: Conn_01x01, Connector_PinHeader_2.54mm:PinHeader_1x01_P2.54mm_Vertical, symbol Connector_Generic:Conn_01x01
- added R6: 75, Resistor_SMD:R_0805_2012Metric_Pad1.15x1.40mm_HandSolder, symbol Device:R_Small
Connections:
- wire segments 51 -> 55
Changed lines of the file:
@@
 	0    1    -1   0
 $EndComp
-Text Label 3500 3400 1    50   ~ 0
+Text Label 3600 3400 1    50   ~ 0
 COMPOSITE
 Text Label 3400 3400 1    50   ~ 0
 LUMA
-Text Label 3600 3400 1    50   ~ 0
+Text Label 3500 3400 1    50   ~ 0
 CHROMA
 $Comp
@@
 L Connector_Generic:Conn_01x01 JAV5
 U 1 1 61F12789
-P 3300 1500
-F 0 "JAV5" V 3350 1800 50  0000 R CNN
-F 1 "Conn_01x01" V 3250 2050 50  0000 R CNN
-F 2 "Connector_PinHeader_2.54mm:PinHeader_1x01_P2.54mm_Vertical" H 3300 1500 50  0001 C CNN
-F 3 "~" H 3300 1500 50  0001 C CNN
-	1    3300 1500
-	0    -1   -1   0
+P 3800 1600
+F 0 "JAV5" V 3850 1900 50  0000 R CNN
+F 1 "Conn_01x01" V 3750 2150 50  0000 R CNN
+F 2 "Connector_PinHeader_2.54mm:PinHeader_1x01_P2.54mm_Vertical" H 3800 1600 50  0001 C CNN
+F 3 "~" H 3800 1600 50  0001 C CNN
+	1    3800 1600
+	0    1    -1   0
 $EndComp
 $Comp
 L Connector_Generic:Conn_01x01 JAV4
 U 1 1 61F127BE
-P 3600 1500
-F 0 "JAV4" V 3650 1200 50  0000 L CNN
-F 1 "Conn_01x01" V 3550 950 50  0000 L CNN
-F 2 "Connector_PinHeader_2.54mm:PinHeader_1x01_P2.54mm_Vertical" H 3600 1500 50  0001 C CNN
-F 3 "~" H 3600 1500 50  0001 C CNN
-	1    3600 1500
-	0    -1   -1   0
+P 3500 1600
+F 0 "JAV4" V 3550 1300 50  0000 L CNN
+F 1 "Conn_01x01" V 3450 1050 50  0000 L CNN
+F 2 "Connector_PinHeader_2.54mm:PinHeader_1x01_P2.54mm_Vertical" H 3500 1600 50  0001 C CNN
+F 3 "~" H 3500 1600 50  0001 C CNN
+	1    3500 1600
+	0    1    -1   0
 $EndComp
 $Comp
 L Device:R_Small R4
 U 1 1 61F12E8F
-P 3300 1900
-F 0 "R4" H 3359 1946 50  0000 L CNN
-F 1 "75" H 3359 1855 50  0000 L CNN
-F 2 "Resistor_SMD:R_0805_2012Metric_Pad1.15x1.40mm_HandSolder" H 3300 1900 50  0001 C CNN
-F 3 "~" H 3300 1900 50  0001 C CNN
-	1    3300 1900
+P 3500 2350
+F 0 "R4" H 3559 2396 50  0000 L CNN
+F 1 "75" H 3559 2305 50  0000 L CNN
+F 2 "Resistor_SMD:R_0805_2012Metric_Pad1.15x1.40mm_HandSolder" H 3500 2350 50  0001 C CNN
+F 3 "~" H 3500 2350 50  0001 C CNN
+	1    3500 2350
 	1    0    0    -1
 $EndComp
@@
 L Device:R_Small R5
 U 1 1 61F12F43
-P 3600 1900
-F 0 "R5" H 3659 1946 50  0000 L CNN
-F 1 "75" H 3659 1855 50  0000 L CNN
-F 2 "Resistor_SMD:R_0805_2012Metric_Pad1.15x1.40mm_HandSolder" H 3600 1900 50  0001 C CNN
-F 3 "~" H 3600 1900 50  0001 C CNN
-	1    3600 1900
-	1    0    0    -1
-$EndComp
-Wire Wire Line
-	3400 2700 3300 2700
-Wire Wire Line
-	3400 2700 3400 2800
-Wire Wire Line
-	3500 2550 3500 3450
-Wire Wire Line
-	3600 2700 3700 2700
-Wire Wire Line
-	3700 2700 3700 2550
-Wire Wire Line
-	3600 2700 3600 2900
+P 3800 2350
+F 0 "R5" H 3859 2396 50  0000 L CNN
+F 1 "75" H 3859 2305 50  0000 L CNN
+F 2 "Resistor_SMD:R_0805_2012Metric_Pad1.15x1.40mm_HandSolder" H 3800 2350 50  0001 C CNN
+F 3 "~" H 3800 2350 50  0001 C CNN
+	1    3800 2350
+	1    0    0    -1
+$EndComp
 $Comp
 L Device:R_POT_TRIM RV2
@@
 F 3 "~" H 3400 5100 50  0001 C CNN
 	1    3400 5100
-	1    0    0    -1
+	1    0    0    1
 $EndComp
 $Comp
@@
 Wire Wire Line
 	2850 3150 2850 2900
-Wire Wire Line
-	2850 2900 3600 2900
-Connection ~ 3600 2900
-Wire Wire Line
-	3600 2900 3600 3450
 $Comp
 L Device:C_Small C2
@@
 Wire Wire Line
 	2850 3450 2850 3350
-Wire Wire Line
-	3500 4200 3500 4100
 $Comp
 L Device:C_Small C3
@@
 	1    0    0    -1
 $EndComp
-Wire Wire Line
-	4100 4700 3600 4700
-Wire Wire Line
-	3600 4700 3600 4100
 Wire Wire Line
 	3400 5400 3400 5200
@@
 	2450 4200 2450 3950
 Wire Wire Line
-	2450 4200 3500 4200
-Wire Wire Line
 	3200 3450 3300 3450
 Wire Wire Line
 	3200 4100 3300 4100
 Wire Wire Line
-	3300 2000 3300 2700
-Wire Wire Line
-	3300 1800 3300 1700
-Wire Wire Line
-	3600 1800 3600 1700
-$Comp
-L Connector_Generic:Conn_01x03 JSELECT1
-U 1 1 61F1E4CA
-P 3600 2350
-F 0 "JSELECT1" V 3566 2162 50  0000 R CNN
-F 1 "Conn_01x03" V 3475 2162 50  0000 R CNN
-F 2 "Connector_PinHeader_2.54mm:PinHeader_1x03_P2.54mm_Horizontal" H 3600 2350 50  0001 C CNN
-F 3 "~" H 3600 2350 50  0001 C CNN
-	1    3600 2350
-	0    1    -1   0
-$EndComp
-Wire Wire Line
-	3600 2000 3600 2550
+	3500 2250 3500 1800
+Wire Wire Line
+	3800 2250 3800 1800
+$Comp
+L Connector_Generic:Conn_01x01 JAV6
+U 1 1 62FE59EE
+P 4150 1900
+F 0 "JAV6" V 4200 1600 50  0000 L CNN
+F 1 "Conn_01x01" V 4100 1350 50  0000 L CNN
+F 2 "Connector_PinHeader_2.54mm:PinHeader_1x01_P2.54mm_Vertical" H 4150 1900 50  0001 C CNN
+F 3 "~" H 4150 1900 50  0001 C CNN
+	1    4150 1900
+	0    -1   -1   0
+$EndComp
+$Comp
+L Device:R_Small R6
+U 1 1 62FE9FFD
+P 4150 2350
+F 0 "R6" H 4209 2396 50  0000 L CNN
+F 1 "75" H 4209 2305 50  0000 L CNN
+F 2 "Resistor_SMD:R_0805_2012Metric_Pad1.15x1.40mm_HandSolder" H 4150 2350 50  0001 C CNN
+F 3 "~" H 4150 2350 50  0001 C CNN
+	1    4150 2350
+	1    0    0    -1
+$EndComp
+Wire Wire Line
+	4150 2250 4150 2100
+Wire Wire Line
+	3400 2600 4150 2600
+Wire Wire Line
+	4150 2600 4150 2450
+Wire Wire Line
+	3400 2600 3400 2800
+$Comp
+L power:PWR_FLAG #FLG0101
+U 1 1 62FEE9FE
+P 6550 5000
+F 0 "#FLG0101" H 6550 5075 50  0001 C CNN
+F 1 "PWR_FLAG" V 6550 5128 50  0000 L CNN
+F 2 "" H 6550 5000 50  0001 C CNN
+F 3 "~" H 6550 5000 50  0001 C CNN
+	1    6550 5000
+	0    -1   -1   0
+$EndComp
+$Comp
+L power:PWR_FLAG #FLG0102
+U 1 1 62FEEA74
+P 6550 5600
+F 0 "#FLG0102" H 6550 5675 50  0001 C CNN
+F 1 "PWR_FLAG" V 6550 5728 50  0000 L CNN
+F 2 "" H 6550 5600 50  0001 C CNN
+F 3 "~" H 6550 5600 50  0001 C CNN
+	1    6550 5600
+	0    -1   -1   0
+$EndComp
+Wire Wire Line
+	6550 5000 6650 5000
+Wire Wire Line
+	6550 5600 6650 5600
+Connection ~ 6650 5600
+Wire Wire Line
+	3500 4700 4100 4700
+Wire Wire Line
+	3500 4100 3500 4700
+Wire Wire Line
+	2450 4200 3600 4200
+Wire Wire Line
+	3600 4200 3600 4100
+Wire Wire Line
+	3500 2800 3800 2800
+Wire Wire Line
+	3500 2800 3500 2900
+Wire Wire Line
+	3800 2450 3800 2800
+Wire Wire Line
+	3600 2700 3500 2700
+Wire Wire Line
+	3500 2700 3500 2450
+Wire Wire Line
+	3600 2700 3600 3450
+Wire Wire Line
+	2850 2900 3500 2900
+Connection ~ 3500 2900
+Wire Wire Line
+	3500 2900 3500 3450
 $EndSCHEMATC
